File: FemtoLCC.kicad_pcb (KiCad board)
At the start: 2 copper layers, 85 x 100 mm, 77 parts, among them J1 Screw_Terminal_01x12, J2 RJHSE508002, J3 SM04B-SRSS-TB, J4 SM04B-SRSS-TB, U1 SN3257QPWRQ1, U10 SN74HC253DR, U11 DRV8874PWPR, U12 6N137, U13 6N137, U2 MCP2562-E-SN, U4 SN74HC253DR, U5 DRV8874PWPR, U6 SN74HC253DR, U7 DRV8874PWPR, U8 SN74HC253DR, U9 DRV8874PWPR

Commit message: Add new routing strategy
Parts:
- removed A1: RaspberryPi_Pico, Module:RaspberryPi_Pico_Common_SMD
- removed U12, U13: 6N137, Package_DIP:DIP-8_W7.62mm_SMDSocket_SmallPads
- added C34: C10u, Capacitor_SMD:C_1206_3216Metric_Pad1.33x1.80mm_HandSolder, F.Cu at (177.5, 77.2)
- added C35: C100n VM, Capacitor_SMD:C_0805_2012Metric_Pad1.18x1.45mm_HandSolder, F.Cu at (193.3, 76.5)
- added C36: C100n, Capacitor_SMD:C_0805_2012Metric_Pad1.18x1.45mm_HandSolder, F.Cu at (175.2, 90.6)
- added C37: C100n, Capacitor_SMD:C_0805_2012Metric_Pad1.18x1.45mm_HandSolder, F.Cu at (112.4, 62.9)
- added C38: C10u VM, Capacitor_SMD:C_1206_3216Metric_Pad1.33x1.80mm_HandSolder, F.Cu at (190.0, 87.1)
- added C39: C100n VM, Capacitor_SMD:C_0805_2012Metric_Pad1.18x1.45mm_HandSolder, F.Cu at (192.5, 86.6)
- added C40: C10u, Capacitor_SMD:C_1206_3216Metric_Pad1.33x1.80mm_HandSolder, F.Cu at (189.2, 100.6)
- added C41: C100n, Capacitor_SMD:C_0805_2012Metric_Pad1.18x1.45mm_HandSolder, F.Cu at (112.4, 68.9)
- added C42: C100n, Capacitor_SMD:C_0805_2012Metric_Pad1.18x1.45mm_HandSolder, F.Cu at (181.6, 93.7)
- added C43: C100n, Capacitor_SMD:C_0805_2012Metric_Pad1.18x1.45mm_HandSolder, F.Cu at (186.7, 157.6)
- added C44: C10u, Capacitor_SMD:C_1206_3216Metric_Pad1.33x1.80mm_HandSolder, F.Cu at (111.6, 75.5)
- added C45: C100n, Capacitor_SMD:C_0805_2012Metric_Pad1.18x1.45mm_HandSolder, F.Cu at (117.0, 75.3)
- added C46: C1u, Capacitor_SMD:C_0805_2012Metric_Pad1.18x1.45mm_HandSolder, F.Cu at (117.0, 78.3)
- added C47: C1u, Capacitor_SMD:C_0805_2012Metric_Pad1.18x1.45mm_HandSolder, F.Cu at (117.0, 81.3)
- added C48: C10u, Capacitor_SMD:C_1206_3216Metric_Pad1.33x1.80mm_HandSolder, F.Cu at (111.6, 78.8)
- added C49: C100n, Capacitor_SMD:C_0805_2012Metric_Pad1.18x1.45mm_HandSolder, F.Cu at (179.6, 102.6)
- added D1: D_Schottky, Diode_SMD:D_SMA_Handsoldering, F.Cu at (193.4, 81.8)
- added D2: D_Schottky, Diode_SMD:D_SMA_Handsoldering, F.Cu at (181.8, 81.8)
- added D3: D10V, Diode_SMD:D_SOD-323_HandSoldering, F.Cu at (209.8, 77.0)
- added D4: LED, LED_SMD:LED_0603_1608Metric, F.Cu at (182.6, 136.7)
- added J10: Conn_01x02, Connector_Phoenix_MC:PhoenixContact_MCV_1,5_2-G-3.5_1x02_P3.50mm_Vertical, F.Cu at (201.6, 75.0)
- added J5: Conn_01x02, TerminalBlock_Phoenix:TerminalBlock_Phoenix_MKDS-1,5-2-5.08_1x02_P5.08mm_Horizontal, F.Cu at (221.8, 93.0)
- added J6: Conn_01x02, TerminalBlock_Phoenix:TerminalBlock_Phoenix_MKDS-1,5-2-5.08_1x02_P5.08mm_Horizontal, F.Cu at (221.8, 112.2)
- added J7: Conn_01x02, TerminalBlock_Phoenix:TerminalBlock_Phoenix_MKDS-1,5-2-5.08_1x02_P5.08mm_Horizontal, F.Cu at (221.8, 131.2)
- added J8: Conn_01x02, TerminalBlock_Phoenix:TerminalBlock_Phoenix_MKDS-1,5-2-5.08_1x02_P5.08mm_Horizontal, F.Cu at (221.8, 150.3)
- added J9: Conn_01x03, Connector_Phoenix_MC:PhoenixContact_MCV_1,5_3-G-3.5_1x03_P3.50mm_Vertical, F.Cu at (172.6, 75.0)
- added P1: USB_C_Plug_USB2.0, Connector_USB:USB_C_Receptacle_G-Switch_GT-USB-7051x, F.Cu at (156.7, 142.0)
- added Q1: AO3401A, Package_TO_SOT_SMD:SOT-23, F.Cu at (206.6, 77.3)
- added R18: R2.2k, Resistor_SMD:R_0402_1005Metric, F.Cu at (174.3, 64.5)
- added R19: R2k 1W, Resistor_SMD:R_2512_6332Metric_Pad1.40x3.35mm_HandSolder, F.Cu at (170.0, 84.3)
- added R20: R2k 1W, Resistor_SMD:R_2512_6332Metric_Pad1.40x3.35mm_HandSolder, F.Cu at (174.8, 84.3)
- added R21: R10k, Resistor_SMD:R_0805_2012Metric_Pad1.20x1.40mm_HandSolder, F.Cu at (178.7, 94.7)
- added R22: R10k, Resistor_SMD:R_0805_2012Metric_Pad1.20x1.40mm_HandSolder, F.Cu at (178.7, 99.3)
- added R23: R5.1k, Resistor_SMD:R_0402_1005Metric, F.Cu at (185.8, 136.7)
- added R24: R, Resistor_SMD:R_1206_3216Metric, F.Cu at (156.2, 50.2)
- added R25: R, Resistor_SMD:R_1206_3216Metric, F.Cu at (156.2, 53.5)
- added R26: R, Resistor_SMD:R_1206_3216Metric, F.Cu at (156.2, 56.8)
- added R27: R, Resistor_SMD:R_1206_3216Metric, F.Cu at (156.2, 60.1)
- added SW1: SW_Push, Capacitor_SMD:C_1206_3216Metric_Pad1.33x1.80mm_HandSolder, F.Cu at (111.6, 82.2)
- added U14: ESP32-C6-WROOM-1, PCM_Espressif:ESP32-C6-WROOM-1, F.Cu at (160.5, 126.5)
- added U15: NCP1117-5.0_SOT223, Package_TO_SOT_SMD:SOT-223-3_TabPin2, F.Cu at (184.0, 88.0)
- added U16: HCPL-2630, Package_DIP:DIP-8_W7.62mm, F.Cu at (168.4, 93.2)
- added U3: MCP23018x-x-SO, Package_SO:SOIC-28W_7.5x17.9mm_P1.27mm, F.Cu at (177.2, 145.6)
- C1: value C100n -> C10u VM; footprint Capacitor_SMD:C_0805_2012Metric_Pad1.18x1.45mm_HandSolder -> Capacitor_SMD:C_1206_3216Metric_Pad1.33x1.80mm_HandSolder
- J1: value Screw_Terminal_01x12 -> UART Header; footprint TerminalBlock_Phoenix:TerminalBlock_Phoenix_MKDS-1,5-12_1x12_P5.00mm_Horizontal -> Connector_PinHeader_2.54mm:PinHeader_1x06_P2.54mm_Vertical
- J3: footprint SM04B_SRSS_TB:CONN_SM04B-SRSS-TB_JST -> Connector_JST:JST_SH_BM04B-SRSS-TB_1x04-1MP_P1.00mm_Vertical
- J4: value SM04B-SRSS-TB -> PMOD; footprint SM04B_SRSS_TB:CONN_SM04B-SRSS-TB_JST -> Connector_PinSocket_2.54mm:PinSocket_2x06_P2.54mm_Horizontal
- JP6: value SolderJumper_2_Open -> Jumper_2_Open; footprint Jumper:SolderJumper-2_P1.3mm_Open_RoundedPad1.0x1.5mm -> TestPoint:TestPoint_2Pads_Pitch2.54mm_Drill0.8mm
- R14: value R10k -> R47k; footprint Resistor_SMD:R_0805_2012Metric_Pad1.20x1.40mm_HandSolder -> Resistor_SMD:R_0402_1005Metric
- R15, R16: value R2k 1W -> R5.1k; footprint Resistor_SMD:R_2512_6332Metric_Pad1.40x3.35mm_HandSolder -> Resistor_SMD:R_0402_1005Metric
- R17: value R10k -> R100; footprint Resistor_SMD:R_0805_2012Metric_Pad1.20x1.40mm_HandSolder -> Resistor_SMD:R_0402_1005Metric
- R2, R3: footprint Resistor_SMD:R_0805_2012Metric_Pad1.20x1.40mm_HandSolder -> Resistor_SMD:R_0402_1005Metric
- R4: value R2.2k -> R47k
- R5: value R2.2k -> R47k; footprint Resistor_SMD:R_0805_2012Metric_Pad1.20x1.40mm_HandSolder -> Resistor_SMD:R_0402_1005Metric
- U1: value SN3257QPWRQ1 -> NCP1117-3.3_SOT223; footprint SN3257QPWRQ1:SOIC_PRQ1_TEX -> Package_TO_SOT_SMD:SOT-223-3_TabPin2
- moved H2 169.1 mm to (220.7, 77.5)
- moved C31 155.2 mm to (213.3, 155.5)
- moved C24 154.5 mm to (213.3, 136.4)
- moved C17 153.8 mm to (213.3, 117.4)
- moved C10 153.2 mm to (213.3, 98.2)
- moved C29 152.6 mm to (214.6, 141.6), turned to 0 degrees
- moved C22 152.3 mm to (214.6, 122.5), turned to 0 degrees
- moved C15 152.1 mm to (214.6, 103.5), turned to 0 degrees
- moved C8 151.8 mm to (214.6, 84.3), turned to 0 degrees
- moved U11 149.3 mm to (212.3, 147.8), turned to 90 degrees
- moved U9 148.8 mm to (212.3, 128.7), turned to 90 degrees
- moved C28 148.6 mm to (217.0, 139.1)
- moved C21 148.3 mm to (217.0, 120.0)
- moved U7 148.3 mm to (212.3, 109.7), turned to 90 degrees
- moved C14 148.1 mm to (217.0, 101.0)
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Connections:
- net /i2c0_scl renamed /i2c_scl
- net /i2c0_sda renamed /i2c_sda
- net Net-(U10-1Y) renamed /Block Driver D/IN1
- net Net-(U10-2Y) renamed /Block Driver D/IN2
- net Net-(U4-1Y) renamed /Block Driver A/IN1
- net Net-(U4-2Y) renamed /Block Driver A/IN2
- net Net-(U6-1Y) renamed /Block Driver B/IN1
- net Net-(U6-2Y) renamed /Block Driver B/IN2
- net Net-(U8-1Y) renamed /Block Driver C/IN1
- net Net-(U8-2Y) renamed /Block Driver C/IN2
- C1 pad 1: +3.3V -> /Power/3.3V_Reg_Vin
- C32 pad 1: +5V -> +3.3V
- C33 pad 1: +5V -> +3.3V
- H1 pad 1: Net-(JP1-B) -> Net-(H1-Pad1)
- H2 pad 1: Net-(JP2-B) -> Net-(H2-Pad1)
- H3 pad 1: Net-(JP3-B) -> Net-(H3-Pad1)
- H4 pad 1: Net-(JP4-B) -> Net-(H4-Pad1)
- J1 pad 1: /raw_dcc_n -> GND
- J1 pad 2: /raw_dcc_p -> unconnected-(J1-Pad2)
- J1 pad 3: /out2_D -> unconnected-(J1-Pad3)
- J1 pad 4: /out1_D -> /uart_rx
- J1 pad 5: /out2_C -> /uart_tx
- J1 pad 6: /out1_C -> (no net)
- J4 pad 1: GND -> /P0
- J4 pad 2: +3.3V -> /P4
- J4 pad 3: /i2c1_sda -> /P1
- J4 pad 4: /i2c1_scl -> /P5
- J4 pad 5: (no net) -> /P2
- J4 pad 6: (no net) -> /P6
- JP6 pad 1: Net-(A1-ADC_VREF) -> Net-(JP6-A)
- JP6 pad 2: +3.3V -> /can-
- R1 pad 1: /can- -> Net-(JP6-A)
- R14 pad 1: /dcc_p -> Net-(P1-SHIELD)
- R14 pad 2: +3.3V -> GND
- R15 pad 1: /raw_dcc_p -> Net-(P1-CC1)
- R15 pad 2: Net-(U12-C) -> GND
- R16 pad 1: /raw_dcc_p -> Net-(P1-CC2)
- R16 pad 2: Net-(U12-C) -> GND
- R17 pad 1: /dcc_n -> Net-(D3-A)
- R17 pad 2: +3.3V -> GND
- R4 pad 2: /i2c1_scl -> Net-(U3-~{RESET})
- R5 pad 2: /i2c1_sda -> /ESP32EN
- U1 pad 1: /adc_sel -> GND
- U1 pad 2: /sense_A -> +3.3V
- U1 pad 3: /sense_B -> /Power/3.3V_Reg_Vin
- U11 pad 10: /out2_D -> /Block Driver D/OUT2
- U11 pad 8: /out1_D -> /Block Driver D/OUT1
- U5 pad 10: /out2_A -> /Block Driver A/OUT2
- U5 pad 8: /out1_A -> /Block Driver A/OUT1
- U7 pad 10: /out2_B -> /Block Driver B/OUT2
- U7 pad 8: /out1_B -> /Block Driver B/OUT1
- U9 pad 10: /out2_C -> /Block Driver C/OUT2
- U9 pad 8: /out1_C -> /Block Driver C/OUT1
Routing:
- net +3.3V: track 421.3 -> 54.6 mm, vias 25 -> 42
- net +5V: track 184.1 -> 25.3 mm, vias 5 -> 4
- net VTRACK: track 104.1 -> 0.00 mm, vias 40 -> 53
- net /raw_dcc_n: track 142.1 -> 49.5 mm, vias 8 -> 0
- net /raw_dcc_p: track 163.8 -> 90.2 mm, vias 4 -> 0
- net /sense_C: track 94.1 -> 22.4 mm, vias 2 -> 0
- net /sense_A: track 66.6 -> 22.4 mm, vias 2 -> 0
- net /sense_B: track 64.7 -> 22.4 mm, vias 2 -> 0
- net /I2Cint: track 0.00 -> 37.6 mm, vias 0 -> 2
- net /nFault_C: track 53.9 -> 17.8 mm
- net /dcc_en_D: track 43.2 -> 7.30 mm
- net /nFault_D: track 52.8 -> 17.8 mm
- net /dir_B: track 26.6 -> 61.0 mm, vias 0 -> 2
- net /dcc_en_A: track 33.5 -> 67.5 mm, vias 0 -> 1
- net Net-(U16-A2): track 0.00 -> 31.4 mm
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- added copper zone on F.Cu, net +3.3V
- added copper zone on In2.Cu, net +3.3V
- added copper zone on F.Cu, net +5V
- added copper zone on In2.Cu, net +5V
- added copper zone on F.Cu, net /Block Driver A/OUT1
- added copper zone on F.Cu, net /Block Driver A/OUT2
- added copper zone on F.Cu, net /Block Driver B/OUT1
- added copper zone on F.Cu, net /Block Driver B/OUT2
- added copper zone on F.Cu, net /Block Driver C/OUT1
- added copper zone on F.Cu, net /Block Driver C/OUT2
- added copper zone on F.Cu, net /Block Driver D/OUT1
- added copper zone on F.Cu, net /Block Driver D/OUT2
- added copper zone on F.Cu, net /Power/3.3V_Reg_Vin
- added copper zone on F.Cu, net /Power/Unfiltered_Vin
- added copper zone on In2.Cu, net /pwr_n
- added copper zone on In2.Cu, net /pwr_p
- added copper zone on In1.Cu, net GND
- added copper zone on B.Cu, net VTRACK
- added copper zone on F.Cu, net VTRACK
- added copper zone on In2.Cu, net VTRACK
- removed copper zone on B.Cu, net GND
Other:
- board size 85 x 100 mm -> 144 x 144.8 mm
- copper layers 2 -> 4
- board text removed: "A+"
- board text removed: "A-"
- board text removed: "B+"
- board text removed: "B-"
- board text removed: "C+"
- board text removed: "C-"
- board text removed: "CAN Term"
- board text removed: "D+"
- board text removed: "D-"
- board text removed: "DCC+"
- board text removed: "DCC-"
- board text removed: "GND"
- board text removed: "LCC JACK"
- board text removed: "Pico LCC Booster"
- board text removed: "QWIIC 0"
- board text removed: "QWIIC 1"
- board text removed: "Rev ${REVISION}"
- board text removed: "VTRACK"
