File: FemtoLCC.kicad_pcb (KiCad board)
At the start: 4 copper layers, 144 x 144.8 mm, 117 parts, among them J1 UART Header, J10 Conn_01x02, J2 RJHSE508002, J3 SM04B-SRSS-TB, J4 PMOD, J5 Conn_01x02, J6 Conn_01x02, J7 Conn_01x02, J8 Conn_01x02, J9 Conn_01x03, P1 USB_C_Plug_USB2.0, Q1 AO3401A, SW1 SW_Push, U1 NCP1117-3.3_SOT223, U10 SN74HC253DR, U11 DRV8874PWPR, U14 ESP32-C6-WROOM-1, U15 NCP1117-5.0_SOT223, U16 HCPL-2630, U2 MCP2562-E-SN, U3 MCP23018x-x-SO, U4 SN74HC253DR, U5 DRV8874PWPR, U6 SN74HC253DR, U7 DRV8874PWPR, U8 SN74HC253DR, U9 DRV8874PWPR

Commit message: preroute
Parts:
- removed JP1, JP2, JP3, JP4: SolderJumper_2_Open, Jumper:SolderJumper-2_P1.3mm_Open_RoundedPad1.0x1.5mm
- removed R24, R25, R26: R, Resistor_SMD:R_1206_3216Metric
- removed U16: HCPL-2630, Package_DIP:DIP-8_W7.62mm
- added U12: HCPL-0630, Package_SO:SOIC-8_3.9x4.9mm_P1.27mm, F.Cu at (171.9, 96.8)
- JP5, R27: moved to B.Cu
- moved JP5 121.6 mm to (162.2, 87.1), turned to 90 degrees
- moved R27 119.1 mm to (214.7, 163.9), turned to 180 degrees
- moved C44 79.3 mm to (153.5, 142.7), turned to 90 degrees
- moved C45 79.0 mm to (193.1, 96.5)
- moved C46 79.0 mm to (193.1, 99.5)
- moved C48 77.9 mm to (156.2, 142.8), turned to -90 degrees
- moved SW1 72.6 mm to (157.6, 138.4), turned to 180 degrees
- moved C37 68.2 mm to (179.7, 73.9), turned to 90 degrees
- moved C47 67.6 mm to (153.4, 138.3), turned to 90 degrees
- moved R15 57.7 mm to (112.9, 90.1)
- moved C3 48.7 mm to (180.4, 108.0)
- moved C2 28.3 mm to (170.5, 104.4), turned to 180 degrees
- moved P1 21.8 mm to (175.3, 130.6)
- moved C40 16.7 mm to (175.7, 90.8), turned to 180 degrees
- moved C36 2.38 mm to (175.2, 93.0)
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Connections:
- H1 pad 1: Net-(H1-Pad1) -> unconnected-(H1-Pad1)_7
- H2 pad 1: Net-(H2-Pad1) -> unconnected-(H2-Pad1)_3
- H3 pad 1: Net-(H3-Pad1) -> unconnected-(H3-Pad1)_8
Routing:
- net /dcc_p: track 171.1 -> 85.5 mm, vias 4 -> 5
- net /dcc_en_A: track 67.5 -> 3.85 mm, vias 1 -> 0
- net /raw_dcc_p: track 90.2 -> 31.4 mm
- net /sense_D: track 74.9 -> 20.5 mm, vias 2 -> 0
- net /dir_B: track 61.0 -> 9.86 mm, vias 2 -> 0
- net /dcc_en_B: track 53.3 -> 4.37 mm, vias 2 -> 0
- net /i2c_scl: track 42.3 -> 0.00 mm, vias 4 -> 0
- net /i2c_sda: track 40.7 -> 0.00 mm, vias 2 -> 0
- net /pwm_D: track 46.7 -> 8.67 mm, vias 2 -> 0
- net /I2Cint: track 37.6 -> 0.00 mm, vias 2 -> 0
- net /dcc_en_C: track 37.1 -> 4.37 mm, vias 2 -> 0
- net /dir_D: track 32.4 -> 9.02 mm, vias 2 -> 1
- net GND: track 158.2 -> 139.8 mm, vias 117 -> 114
- net /pwr_p: track 0.00 -> 16.9 mm
- net /pwr_n: track 0.00 -> 16.9 mm
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Other:
- board size 144 x 144.8 mm -> 76.2 x 95.2 mm
