File: FemtoLCC.kicad_sch (KiCad schematic)
At the start: 24 parts, among them J1 Screw_Terminal_01x12, J2 RJHSE508002, J3 SM04B-SRSS-TB, J4 PMOD, U14 ESP32-C6-WROOM-1, U2 MCP2562-E-SN, U3 MCP23018x-x-SO

Commit message: Add new routing strategy
Parts:
- removed J1: Screw_Terminal_01x12, TerminalBlock_Phoenix:TerminalBlock_Phoenix_MKDS-1,5-12_1x12_P5.00mm_Horizontal, symbol Connector:Screw_Terminal_01x12
- removed JP1, JP2, JP3, JP4: SolderJumper_2_Open, Jumper:SolderJumper-2_P1.3mm_Open_RoundedPad1.0x1.5mm, symbol Jumper:SolderJumper_2_Open
- added C32, C33, C43, C45: C100n, Capacitor_SMD:C_0805_2012Metric_Pad1.18x1.45mm_HandSolder, symbol Device:C
- added C44, C48: C10u, Capacitor_SMD:C_1206_3216Metric_Pad1.33x1.80mm_HandSolder, symbol Device:C
- added C46, C47: C1u, Capacitor_SMD:C_0805_2012Metric_Pad1.18x1.45mm_HandSolder, symbol Device:C
- added D4: LED, LED_SMD:LED_0603_1608Metric, symbol Device:LED
- added J1: UART Header, Connector_PinHeader_2.54mm:PinHeader_1x06_P2.54mm_Vertical, symbol KiCadLibMRR:UART-Header
- added JP6: Jumper_2_Open, TestPoint:TestPoint_2Pads_Pitch2.54mm_Drill0.8mm, symbol Jumper:Jumper_2_Open
- added P1: USB_C_Plug_USB2.0, Connector_USB:USB_C_Receptacle_G-Switch_GT-USB-7051x, symbol Connector:USB_C_Receptacle_USB2.0_14P
- added R14: R47k, Resistor_SMD:R_0402_1005Metric, symbol Device:R
- added R15, R16, R23: R5.1k, Resistor_SMD:R_0402_1005Metric, symbol Device:R
- added R24, R25, R26, R27: R, Resistor_SMD:R_1206_3216Metric, symbol Device:R
- added SW1: SW_Push, Capacitor_SMD:C_1206_3216Metric_Pad1.33x1.80mm_HandSolder, symbol Switch:SW_Push_45deg
- J3: footprint SM04B_SRSS_TB:CONN_SM04B-SRSS-TB_JST -> Connector_JST:JST_SH_BM04B-SRSS-TB_1x04-1MP_P1.00mm_Vertical
- J4: footprint (none) -> Connector_PinSocket_2.54mm:PinSocket_2x06_P2.54mm_Horizontal
- R1: now fitted
- R18, R2, R3, R5: footprint Resistor_SMD:R_0805_2012Metric_Pad1.20x1.40mm_HandSolder -> Resistor_SMD:R_0402_1005Metric
Connections:
- net +3.3V: now also J4.11 (3V3), C32.1, C33.1, C43.1, C44.1, C45.1, C47.2, C48.1, R23.1; no longer J4.6 (3V3)
- net GND: now also J4.10 (GND), J4.9 (GND), C32.2, C33.2, C43.2, C44.2, C45.2, C46.1, C47.1, C48.2, J1.1 (GND), P1.A1 (GND), P1.A12 (GND), P1.B1 (GND), P1.B12 (GND), R14.2, R15.2, R16.2, R24.2, R25.2, R26.2, R27.2, SW1.1; no longer J4.11 (GND), J4.5 (GND)
- net P1: now also J4.3 (IO1); no longer J4.2 (IO1)
- net P2: now also J4.5 (IO2); no longer J4.3 (IO2)
- net P3: now also J4.7 (IO3); no longer J4.4 (IO3)
- net P4: now also J4.2 (IO4); no longer J4.7 (IO4)
- net P5: now also J4.4 (IO5); no longer J4.8 (IO5)
- net P6: now also J4.6 (IO6); no longer J4.9 (IO6)
- net P7: now also J4.8 (IO7); no longer J4.10 (IO7)
- net can-: now also JP6.2 (B); no longer R1.1
- net dcc_en_C: now also U3.5 (GPB2); no longer U3.6 (GPB3)
- net dcc_en_D: now also U3.6 (GPB3); no longer U3.5 (GPB2)
- net uart_rx: now also J1.4 (RX)
- net uart_tx: now also J1.5 (TX)
- net usb_d+: now also P1.A6 (D+), P1.B6 (D+)
- net usb_d-: now also P1.A7 (D-), P1.B7 (D-)
- net at H2.1: now also R25.1
- net at H4.1: now also R27.1
- net at H1.1: now also R24.1
- net ESP32EN: now reaches R5.2, U14.3 (EN/CHIP_PU)
- net ESP32EN: now also C46.2, SW1.2
- net at H3.1: now also R26.1
- net led: no longer names the net of U3.7 (GPB4)
- net led: now also D4.1 (K)
- new net: D4.2 (A), R23.2
- new net: P1.B5 (CC2), R16.1
- new net: P1.S1 (SHIELD), R14.1
- new net: JP6.1 (A), R1.1
- new net: P1.A5 (CC1), R15.1
- new net VBUS: P1.A4 (VBUS), P1.A9 (VBUS), P1.B4 (VBUS), P1.B9 (VBUS)
Other:
- sheet Block Driver A ports: added none; removed OUT1, OUT2
- sheet Block Driver B ports: added none; removed OUT1, OUT2
- sheet Block Driver C ports: added none; removed OUT1, OUT2
- sheet Block Driver D ports: added none; removed OUT1, OUT2
- moved on the sheet: C2, C3, J2A, J2B, J3, J4, JP5, R18, R2, R3, R4, U2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
