File: FemtoLCC.kicad_sch (KiCad schematic)
At the start: 40 parts, among them J1 UART Header, J2 RJHSE508002, J3 SM04B-SRSS-TB, J4 PMOD, P1 USB_C_Plug_USB2.0, SW1 SW_Push, U14 ESP32-C6-WROOM-1, U2 MCP2562-E-SN, U3 MCP23018x-x-SO

Commit message: preroute
Parts:
- removed R24, R25, R26: R, Resistor_SMD:R_1206_3216Metric, symbol Device:R
Connections:
- no-connect marks 1 -> 4
