File: FemtoLCC.kicad_sch (KiCad schematic)
At the start: 37 parts, among them J1 UART Header, J2 RJHSE508002, J3 SM04B-SRSS-TB, J4 PMOD, P1 USB_C_Plug_USB2.0, SW1 SW_Push, U14 ESP32-C6-WROOM-1, U2 MCP2562-E-SN, U3 MCP23018x-x-SO

Commit message: Add fab pipeline, firmware, docs site, and tooling
- Makefile: kicad-cli gerber/drill/BOM/CPL/render exports, ERC/DRC, Hugo
  docs build, and firmware delegation to software/Makefile
- software/: ESP32-C6 Arduino firmware (channels, DCC source, expander,
  LCC traction, occupancy, throttle)
- site/: Hugo documentation site with GitHub Pages workflow
- tools/: BOM/CPL to JLCPCB converters, LCSC part map, stock checker
- production/: gerber bundle, board renders, ordering README
- .gitignore: firmware build output, __pycache__, upload staging,
  Hugo output, ERC/DRC reports; un-ignore tools/lcsc-parts.csv
- KiCad board, schematic, and DRV8874 footprint updates

Co-Authored-By: Claude Fable 5.1 <noreply@anthropic.com>
Claude-Session: https://claude.ai/code/session_01YbF1hVKFHpjgKwz3CaXtPo
Parts:
- added R24: R2.2k, Resistor_SMD:R_0402_1005Metric, symbol Device:R
- SW1: footprint Capacitor_SMD:C_1206_3216Metric_Pad1.33x1.80mm_HandSolder -> Button_Switch_SMD:SW_Push_1P1T_XKB_TS-1187A
Connections:
- net GND: now also R24.2; no longer SW1.1
- new net: R24.1, SW1.1
Changed lines of the file:
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@@
 	(wire
 		(pts
+			(xy 132.08 26.67) (xy 137.16 26.67)
+		)
+		(stroke
+			(width 0)
+			(type default)
+		)
+	)
+	(wire
+		(pts
 			(xy 101.6 90.17) (xy 101.6 77.47)
 		)
@@
 	(wire
 		(pts
-			(xy 135.89 26.67) (xy 137.16 26.67)
-		)
-		(stroke
-			(width 0)
-			(type default)
-		)
-	)
-	(wire
-		(pts
 			(xy 64.77 154.94) (xy 64.77 139.7)
 		)
@@
 	)
 	(symbol
-		(lib_id "power:GND")
-		(at 135.89 26.67 0)
-		(unit 1)
-		(body_style 1)
-		(exclude_from_sim no)
-		(in_bom yes)
-		(on_board yes)
-		(in_pos_files yes)
-		(dnp no)
-		(property "Reference" "#PWR072"
-			(at 135.89 33.02 0)
-			(hide yes)
-			(show_name no)
-			(do_not_autoplace no)
-			(effects
-				(font
-					(size 1.27 1.27)
-				)
-			)
-		)
-		(property "Value" "GND"
-			(at 135.89 30.48 0)
-			(show_name no)
-			(do_not_autoplace no)
-			(effects
-				(font
-					(size 1.27 1.27)
-				)
-			)
-		)
-		(property "Footprint" ""
-			(at 135.89 26.67 0)
-			(hide yes)
-			(show_name no)
-			(do_not_autoplace no)
-			(effects
-				(font
-					(size 1.27 1.27)
-				)
-			)
-		)
-		(property "Datasheet" ""
-			(at 135.89 26.67 0)
-			(hide yes)
-			(show_name no)
-			(do_not_autoplace no)
-			(effects
-				(font
-					(size 1.27 1.27)
-				)
-			)
-		)
-		(property "Description" "Power symbol creates a global label with name \"GND\" , ground"
-			(at 135.89 26.67 0)
-			(hide yes)
-			(show_name no)
-			(do_not_autoplace no)
-			(effects
-				(font
-					(size 1.27 1.27)
-				)
-			)
-		)
-		(pin "1"
-		)
-		(instances
-			(project "FemtoLCC"
-				(path "/52455d2f-97dd-4d4c-8361-4f75b5320576"
-					(reference "#PWR072")
-					(unit 1)
-				)
-			)
-		)
-	)
-	(symbol
 		(lib_id "power:+3.3V")
 		(at 137.16 68.58 0)
@@
 	(symbol
 		(lib_id "Device:R")
+		(at 132.08 30.48 0)
+		(mirror y)
+		(unit 1)
+		(body_style 1)
+		(exclude_from_sim no)
+		(in_bom yes)
+		(on_board yes)
+		(in_pos_files yes)
+		(dnp no)
+		(property "Reference" "R24"
+			(at 129.54 29.2099 0)
+			(show_name no)
+			(do_not_autoplace no)
+			(effects
+				(font
+					(size 1.27 1.27)
+				)
+				(justify left)
+			)
+		)
+		(property "Value" "R2.2k"
+			(at 129.54 31.7499 0)
+			(show_name no)
+			(do_not_autoplace no)
+			(effects
+				(font
+					(size 1.27 1.27)
+				)
+				(justify left)
+			)
+		)
+		(property "Footprint" "Resistor_SMD:R_0402_1005Metric"
+			(at 133.858 30.48 90)
+			(hide yes)
+			(show_name no)
+			(do_not_autoplace no)
+			(effects
+				(font
+					(size 1.27 1.27)
+				)
+			)
+		)
+		(property "Datasheet" ""
+			(at 132.08 30.48 0)
+			(hide yes)
+			(show_name no)
+			(do_not_autoplace no)
+			(effects
+				(font
+					(size 1.27 1.27)
+				)
+			)
+		)
+		(property "Description" "Resistor"
+			(at 132.08 30.48 0)
+			(hide yes)
+			(show_name no)
+			(do_not_autoplace no)
+			(effects
+				(font
+					(size 1.27 1.27)
+				)
+			)
+		)
+		(property "Manufacturer Part Number" "ERJ6ENF4702V"
+			(at 132.08 30.48 0)
+			(hide yes)
+			(show_name no)
+			(do_not_autoplace no)
+			(effects
+				(font
+					(size 1.27 1.27)
+				)
+			)
+		)
+		(property "MANUFACTURER" "Panasonic"
+			(at 132.08 30.48 0)
+			(hide yes)
+			(show_name no)
+			(do_not_autoplace no)
+			(effects
+				(font
+					(size 1.27 1.27)
+				)
+			)
+		)
+		(pin "1"
+		)
+		(pin "2"
+		)
+		(instances
+			(project "FemtoLCC"
+				(path "/52455d2f-97dd-4d4c-8361-4f75b5320576"
+					(reference "R24")
+					(unit 1)
+				)
+			)
+		)
+	)
+	(symbol
+		(lib_id "Device:R")
 		(at 223.52 55.88 0)
 		(unit 1)
@@
 			)
 		)
-		(property "Footprint" "Capacitor_SMD:C_1206_3216Metric_Pad1.33x1.80mm_HandSolder"
+		(property "Footprint" "Button_Switch_SMD:SW_Push_1P1T_XKB_TS-1187A"
 			(at 139.7 29.21 0)
 			(hide yes)
@@
 					(unit 1)
 				)
+			)
+		)
+	)
+	(symbol
+		(lib_id "power:GND")
+		(at 132.08 34.29 0)
+		(unit 1)
+		(body_style 1)
+		(exclude_from_sim no)
+		(in_bom yes)
+		(on_board yes)
+		(in_pos_files yes)
+		(dnp no)
+		(property "Reference" "#PWR072"
+			(at 132.08 40.64 0)
+			(hide yes)
+			(show_name no)
+			(do_not_autoplace no)
+			(effects
+				(font
+					(size 1.27 1.27)
+				)
+			)
+		)
+		(property "Value" "GND"
+			(at 132.08 38.1 0)
+			(show_name no)
+			(do_not_autoplace no)
+			(effects
+				(font
+					(size 1.27 1.27)
+				)
+			)
+		)
+		(property "Footprint" ""
+			(at 132.08 34.29 0)
+			(hide yes)
+			(show_name no)
+			(do_not_autoplace no)
+			(effects
+				(font
+					(size 1.27 1.27)
+				)
+			)
+		)
+		(property "Datasheet" ""
+			(at 132.08 34.29 0)
+			(hide yes)
+			(show_name no)
+			(do_not_autoplace no)
+			(effects
+				(font
+					(size 1.27 1.27)
+				)
+			)
+		)
+		(property "Description" "Power symbol creates a global label with name \"GND\" , ground"
+			(at 132.08 34.29 0)
+			(hide yes)
+			(show_name no)
+			(do_not_autoplace no)
+			(effects
+				(font
+					(size 1.27 1.27)
+				)
+			)
+		)
+		(pin "1"
+		)
+		(instances
+			(project "FemtoLCC"
+				(path "/52455d2f-97dd-4d4c-8361-4f75b5320576"
+					(reference "#PWR072")
+					(unit 1)
+				)

Commit message: Fix product name in schematic title blocks
The title block on all four sheets read "Femto LCC Booster" with a space,
against "FemtoLCC" everywhere else including the silkscreen. Title text
only; no change to symbols, nets or connectivity.

Co-Authored-By: Claude Opus 5 (1M context) <noreply@anthropic.com>
Other:
- title: Femto LCC Booster -> FemtoLCC Booster
Changed lines of the file:
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@@
 	(paper "USLetter")
 	(title_block
-		(title "Femto LCC Booster")
+		(title "FemtoLCC Booster")
 		(date "2025-10-31")
 		(rev "1")
