File: block_driver.kicad_sch (KiCad schematic)
At the start: 11 parts, among them U4 SN74HC253DR, U5 DRV8874PWPR

Commit message: Add new routing strategy
Parts:
- added J5: Conn_01x02, TerminalBlock_Phoenix:TerminalBlock_Phoenix_MKDS-1,5-2-5.08_1x02_P5.08mm_Horizontal, symbol Connector_Generic:Conn_01x02
Connections:
- net OUT1: now also J5.1 (Pin_1)
- net OUT2: now also J5.2 (Pin_2)
- net IN1: now reaches U4.7 (1Y), U5.1 (EN_IN1)
- net IN2: now reaches U4.9 (2Y), U5.2 (PH_IN2)
Other:
- moved on the sheet: C4, C5, R6
