File: dcc_isolator.kicad_sch (KiCad schematic)
At the start: 7 parts, among them U16 HCPL-2630

Commit message: Add new routing strategy
Parts:
- added C49: C100n, Capacitor_SMD:C_0805_2012Metric_Pad1.18x1.45mm_HandSolder, symbol Device:C
- added J9: Conn_01x03, Connector_Phoenix_MC:PhoenixContact_MCV_1,5_3-G-3.5_1x03_P3.50mm_Vertical, symbol Connector_Generic:Conn_01x03
Connections:
- net +3.3V: now also C49.1
- net GND: now also C49.2, J9.2 (Pin_2)
- net raw_dcc_n: now also J9.3 (Pin_3)
- net raw_dcc_p: now also J9.1 (Pin_1)
- net at R20.2, U16.4 (A2): now also R19.2, U16.2 (C1)
Other:
- moved on the sheet: C36, C42, R19, R20, R21, R22, U16
