File: dcc_isolator.kicad_sch (KiCad schematic)
At the start: 9 parts, among them J9 Conn_01x03, U12 HCPL-0630

Commit message: Fix product name in schematic title blocks
The title block on all four sheets read "Femto LCC Booster" with a space,
against "FemtoLCC" everywhere else including the silkscreen. Title text
only; no change to symbols, nets or connectivity.

Co-Authored-By: Claude Opus 5 (1M context) <noreply@anthropic.com>
Other:
- title: Femto LCC Booster -> FemtoLCC Booster
Changed lines of the file:
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@@
 	(paper "USLetter")
 	(title_block
-		(title "Femto LCC Booster")
+		(title "FemtoLCC Booster")
 		(date "2025-10-31")
 		(rev "1")
